Commit message: fix urdf v2

File: src/msr_description/urdf/mecanum_wheel.xacro (robot description, xacro)
@@ -32,9 +32,8 @@
       <xacro:cylinder_inertia mass="0.25" radius="0.04" length="0.035"/>
     </link>
-    <joint name="${name}_joint" type="continuous">
+    <joint name="${name}_joint" type="fixed">
       <parent link="${parent}"/>
       <child link="${name}"/>
       <origin xyz="${xyz}" rpy="${rpy}"/>
-      <axis xyz="0 0 1"/>
     </joint>
   </xacro:macro>

File: src/msr_description/urdf/msr_robot.urdf.xacro (robot description, xacro)
@@ -6,11 +6,5 @@
   <xacro:include filename="$(find msr_description)/urdf/sensors.xacro"/>
   <xacro:include filename="$(find msr_description)/urdf/arm_mg996r.xacro"/>
-  <!-- base footprint -->
-  <link name="base_footprint"/>
-  <joint name="base_footprint_to_base_link" type="fixed">
-    <parent link="base_footprint"/>
-    <child link="base_link"/>
-    <origin xyz="0 0 0.08" rpy="0 0 0"/>
-  </joint>
+  <!-- base_link is now the root link; base_footprint is omitted for correct TF hierarchy -->
   <xacro:msr_chassis/>
   <!-- 80mm wheels, visual mecanum-like, physics handled in Gazebo SDF by DiffDrive for Day 1 -->
